Commit message: solve a error

File: my_robot/urdf/my_robot.xacro (robot description, xacro)
@@ -132,23 +132,7 @@
     		<axis xyz="0 1 0" rpy="0 0 0"/>
   	</joint>
-  	<link name="camera_link_optical">
-		<!--<inertial>
-      			<mass value="0.1"/>
-      			<origin xyz="0 0 0" rpy="0 0 0"/>
-      			<box_inertia m="0.1" x="0.05" y="0.05" z="0.05"/>
-      			<inertia
-          			ixx="1e-6" ixy="0" ixz="0"
-          			iyy="1e-6" iyz="0"
-          			izz="1e-6"/>
-    		</inertial>
-		<visual name='camera_visual_optical'>
-      			<origin xyz="0 0 0" rpy="0 -1 0"/>
-      			<geometry>
-        			<box size=".05 .05 .1"/>
-      			</geometry>
-    		</visual>-->
-  	</link>
+  	<link name="camera_link_optical"></link>
   	<joint name="camera_optical_joint" type="fixed">
-    		<origen xyz="0 0 0" rpy="-1.5707 0 -1.5707" />
+    		<origin xyz="0 0 0" rpy="-1.5707 0 -1.5707" />
     		<parent link="camera_link"/>
     		<child link="camera_link_optical" />
